Commit message: New naming of package, added -support

File: motoman_gp400_support/urdf/gp400.xacro (robot description, xacro)
@@ -1,5 +1,5 @@
 <?xml version="1.0" ?>
 <robot name="motoman_gp400" xmlns:xacro="http://ros.org/wiki/xacro">
-        <xacro:include filename="$(find motoman_gp400)/urdf/gp400_macro.xacro" />
+        <xacro:include filename="$(find motoman_gp400_support)/urdf/gp400_macro.xacro" />
         <xacro:motoman_gp400 prefix=""/>
 </robot>

File: motoman_gp400_support/urdf/gp400_macro.xacro (robot description, xacro)
@@ -5,7 +5,4 @@
         <material name="${prefix}Yaskawa_blue">
             <color rgba="0.12941 0.14902 0.74902 1" />
-        </material>
-        <material name="${prefix}NOV_red">
-            <color rgba="0.8 0.1412 0.1725 1" />
         </material>
         <material name="${prefix}Collision_yellow">
@@ -19,11 +16,11 @@
             <visual>
                 <geometry>
-                    <mesh filename="package://motoman_gp400/meshes/visual/GP400_BASE_AXIS.stl"/>
-                </geometry>
-                <material name="${prefix}NOV_red"/>
-            </visual>
-            <collision>
-                <geometry>
-                    <mesh filename="package://motoman_gp400/meshes/visual/GP400_BASE_AXIS.stl"/>
+                    <mesh filename="package://motoman_gp400_support/meshes/visual/GP400_BASE_AXIS.stl"/>
+                </geometry>
+                <material name="${prefix}Yaskawa_blue"/>
+            </visual>
+            <collision>
+                <geometry>
+                    <mesh filename="package://motoman_gp400_support/meshes/visual/GP400_BASE_AXIS.stl"/>
                 </geometry>
                 <material name="${prefix}Collision_yellow"/>
@@ -33,11 +30,11 @@
             <visual>
                 <geometry>
-                    <mesh filename="package://motoman_gp400/meshes/visual/GP400_S_AXIS.stl"/>
-                </geometry>
-                <material name="${prefix}NOV_red"/>
-            </visual>
-            <collision>
-                <geometry>
-                    <mesh filename="package://motoman_gp400/meshes/visual/GP400_S_AXIS.stl"/>
+                    <mesh filename="package://motoman_gp400_support/meshes/visual/GP400_S_AXIS.stl"/>
+                </geometry>
+                <material name="${prefix}Yaskawa_blue"/>
+            </visual>
+            <collision>
+                <geometry>
+                    <mesh filename="package://motoman_gp400_support/meshes/visual/GP400_S_AXIS.stl"/>
                 </geometry>
                 <material name="${prefix}Collision_yellow"/>
@@ -47,11 +44,11 @@
             <visual>
                 <geometry>
-                    <mesh filename="package://motoman_gp400/meshes/visual/GP400_L_AXIS.stl"/>
-                </geometry>
-                <material name="${prefix}NOV_red"/>
-            </visual>
-            <collision>
-                <geometry>
-                    <mesh filename="package://motoman_gp400/meshes/collision/GP400_L_AXIS.stl"/>
+                    <mesh filename="package://motoman_gp400_support/meshes/visual/GP400_L_AXIS.stl"/>
+                </geometry>
+                <material name="${prefix}Yaskawa_blue"/>
+            </visual>
+            <collision>
+                <geometry>
+                    <mesh filename="package://motoman_gp400_support/meshes/collision/GP400_L_AXIS.stl"/>
                 </geometry>
                 <material name="${prefix}Collision_yellow"/>
@@ -61,11 +58,11 @@
             <visual>
                 <geometry>
-                    <mesh filename="package://motoman_gp400/meshes/visual/GP400_U_AXIS.stl"/>
-                </geometry>
-                <material name="${prefix}NOV_red"/>
-            </visual>
-            <collision>
-                <geometry>
-                    <mesh filename="package://motoman_gp400/meshes/collision/GP400_U_AXIS.stl"/>
+                    <mesh filename="package://motoman_gp400_support/meshes/visual/GP400_U_AXIS.stl"/>
+                </geometry>
+                <material name="${prefix}Yaskawa_blue"/>
+            </visual>
+            <collision>
+                <geometry>
+                    <mesh filename="package://motoman_gp400_support/meshes/collision/GP400_U_AXIS.stl"/>
                 </geometry>
                 <material name="${prefix}Collision_yellow"/>
@@ -75,11 +72,11 @@
             <visual>
                 <geometry>
-                    <mesh filename="package://motoman_gp400/meshes/visual/GP400_R_AXIS.stl"/>
-                </geometry>
-                <material name="${prefix}NOV_red"/>
-            </visual>
-            <collision>
-                <geometry>
-                    <mesh filename="package://motoman_gp400/meshes/collision/GP400_R_AXIS.stl"/>
+                    <mesh filename="package://motoman_gp400_support/meshes/visual/GP400_R_AXIS.stl"/>
+                </geometry>
+                <material name="${prefix}Yaskawa_blue"/>
+            </visual>
+            <collision>
+                <geometry>
+                    <mesh filename="package://motoman_gp400_support/meshes/collision/GP400_R_AXIS.stl"/>
                 </geometry>
                 <material name="${prefix}Collision_yellow"/>
@@ -89,11 +86,11 @@
             <visual>
                 <geometry>
-                    <mesh filename="package://motoman_gp400/meshes/visual/GP400_B_AXIS.stl"/>
-                </geometry>
-                <material name="${prefix}NOV_red"/>
-            </visual>
-            <collision>
-                <geometry>
-                    <mesh filename="package://motoman_gp400/meshes/collision/GP400_B_AXIS.stl"/>
+                    <mesh filename="package://motoman_gp400_support/meshes/visual/GP400_B_AXIS.stl"/>
+                </geometry>
+                <material name="${prefix}Yaskawa_blue"/>
+            </visual>
+            <collision>
+                <geometry>
+                    <mesh filename="package://motoman_gp400_support/meshes/collision/GP400_B_AXIS.stl"/>
                 </geometry>
                 <material name="${prefix}Collision_yellow"/>
@@ -103,12 +100,12 @@
             <visual>
                 <geometry>
-                    <mesh filename="package://motoman_gp400/meshes/visual/GP400_T_AXIS.stl"/>
-                </geometry>
-                <!-- <material name="${prefix}NOV_red"/> -->
+                    <mesh filename="package://motoman_gp400_support/meshes/visual/GP400_T_AXIS.stl"/>
+                </geometry>
+                <!-- <material name="${prefix}Yaskawa_blue"/> -->
                 <material name="${prefix}Component_grey"/>
             </visual>
             <collision>
                 <geometry>
-                    <mesh filename="package://motoman_gp400/meshes/collision/GP400_T_AXIS.stl"/>
+                    <mesh filename="package://motoman_gp400_support/meshes/collision/GP400_T_AXIS.stl"/>
                 </geometry>
                 <material name="${prefix}Collision_yellow"/>
@@ -119,13 +116,13 @@
             <visual>
                 <geometry>
-                    <mesh filename="package://motoman_gp400/meshes/visual/GP400_LINK_A_AXIS (Origin in upper joint).stl"/>
-                    <!-- <mesh filename="package://motoman_gp400/meshes/visual/GP400_LINK_A_AXIS.stl"/> -->
-                </geometry>
-                <material name="${prefix}NOV_red"/>
-            </visual>
-            <collision>
-                <geometry>
-                    <mesh filename="package://motoman_gp400/meshes/collision/GP400_LINK_A_AXIS (Origin in upper joint).stl"/>
-                    <!-- <mesh filename="package://motoman_gp400/meshes/collision/GP400_LINK_A_AXIS.stl"/> -->
+                    <!-- <mesh filename="package://motoman_gp400_support/meshes/visual/GP400_LINK_A_AXIS (Origin in upper joint).stl"/> -->
+                    <mesh filename="package://motoman_gp400_support/meshes/visual/GP400_LINK_A_AXIS.stl"/>
+                </geometry>
+                <material name="${prefix}Yaskawa_blue"/>
+            </visual>
+            <collision>
+                <geometry>
+                    <!-- <mesh filename="package://motoman_gp400_support/meshes/collision/GP400_LINK_A_AXIS (Origin in upper joint).stl"/> -->
+                    <mesh filename="package://motoman_gp400_support/meshes/collision/GP400_LINK_A_AXIS.stl"/>
                 </geometry>
                 <material name="${prefix}Collision_yellow"/>
@@ -136,11 +133,11 @@
             <visual>
                 <geometry>
-                    <mesh filename="package://motoman_gp400/meshes/visual/GP400_LINK_B_AXIS.stl"/>
-                </geometry>
-                <material name="${prefix}NOV_red"/>
-            </visual>
-            <collision>
-                <geometry>
-                    <mesh filename="package://motoman_gp400/meshes/visual/GP400_LINK_B_AXIS.stl"/>
+                    <mesh filename="package://motoman_gp400_support/meshes/visual/GP400_LINK_B_AXIS.stl"/>
+                </geometry>
+                <material name="${prefix}Yaskawa_blue"/>
+            </visual>
+            <collision>
+                <geometry>
+                    <mesh filename="package://motoman_gp400_support/meshes/visual/GP400_LINK_B_AXIS.stl"/>
                 </geometry>
                 <material name="${prefix}Collision_yellow"/>
@@ -151,12 +148,12 @@
             <visual>
                 <geometry>
-                    <mesh filename="package://motoman_gp400/meshes/visual/GP400_BALANCER_1_AXIS.stl"/>
-                </geometry>
-                <!-- <material name="${prefix}NOV_red"/> -->
+                    <mesh filename="package://motoman_gp400_support/meshes/visual/GP400_BALANCER_1_AXIS.stl"/>
+                </geometry>
+                <!-- <material name="${prefix}Yaskawa_blue"/> -->
                 <material name="${prefix}Component_grey"/>
             </visual>
             <collision>
                 <geometry>
-                    <mesh filename="package://motoman_gp400/meshes/collision/GP400_BALANCER_1_AXIS.stl"/>
+                    <mesh filename="package://motoman_gp400_support/meshes/collision/GP400_BALANCER_1_AXIS.stl"/>
                 </geometry>
                 <material name="${prefix}Collision_yellow"/>
@@ -164,6 +161,5 @@
         </link>
         <link name="${prefix}tool0"/>
-        <link name="${prefix}fakelinkA"/>
-        <link name="${prefix}fakelinkJ3"/>
+        <link name="${prefix}fakelink"/>
         <!-- End of Link List -->
         <!-- Joint List -->
@@ -185,19 +181,14 @@
         </joint>
         <!-- U-Axis -->
-        <joint name="${prefix}fakelinkJ3_to_joint_2" type="revolute">
+        <joint name="${prefix}joint_3" type="revolute">
             <parent link="${prefix}link_2"/>
-            <child link="${prefix}fakelinkJ3"/>
+            <child link="${prefix}link_3"/>
             <origin xyz="0.000 0.000 1.050" rpy="0 0 0" />
-            <axis xyz="0 1 0" />
-            <mimic joint="${prefix}joint_2" multiplier="-1" offset="${radians(0)}"/>
-            <limit lower="${radians(-180)}" upper="${radians(180)}" velocity="1.69" effort="0"/>
-        </joint>
-        <!-- U-Axis -->
-        <joint name="${prefix}joint_3" type="revolute">
-            <parent link="${prefix}fakelinkJ3"/>
-            <child link="${prefix}link_3"/>
-            <origin xyz="0.000 0.000 0.000" rpy="0 0 0" />
-            <axis xyz="0 -1 0" />
-            <limit lower="${radians(-52)}" upper="${radians(61)}" velocity="1.69" effort="0"/>
+            <axis xyz="0 -1 0" />
+            <!-- <limit lower="${radians(-18)}" upper="${radians(113)}" velocity="1.69" effort="0"/> -->
+            <!-- <limit lower="${radians(-52)}" upper="${radians(61)}" velocity="1.69" effort="0"/> -->
+            <limit lower="${radians(-61)}" upper="${radians(17)}" velocity="1.69" effort="0"/>
+            <!-- Lower = -113 + 61 -->
+            <!-- Upper = 61-->
         </joint>
         <!-- R-Axis -->
@@ -207,5 +198,6 @@
             <origin xyz="1.31772 0.000 0.250" rpy="0 0 0" />
             <axis xyz="-1 0 0" />
-            <limit lower="${radians(-360)}" upper="${radians(360)}" velocity="1.40" effort="0"/>
+            <!-- <limit lower="${radians(-360)}" upper="${radians(360)}" velocity="1.40" effort="0"/> -->
+            <limit lower="${radians(-120)}" upper="${radians(120)}" velocity="1.40" effort="0"/>
         </joint>
         <!-- B-Axis -->
@@ -223,5 +215,6 @@
             <origin xyz="0.266 0.000 0.000" rpy="0 0 0" />
             <axis xyz="-1 0 0" />
-            <limit lower="${radians(-360)}" upper="${radians(360)}" velocity="3.00" effort="0"/>
+            <!-- <limit lower="${radians(-360)}" upper="${radians(360)}" velocity="3.00" effort="0"/> -->
+            <limit lower="${radians(-120)}" upper="${radians(120)}" velocity="3.00" effort="0"/>
         </joint>
         <!-- EOAT -->
@@ -231,31 +224,50 @@
             <child link="${prefix}tool0"/>
         </joint>
+        <!-- Fakelinke for Balancer B -->
+        <joint name="${prefix}link1_adjustment" type="revolute">
+            <origin xyz="0.400 0.000 0.7555" rpy="0 0 0"/>
+            <parent link="${prefix}link_1"/>
+            <child link="${prefix}fakelink"/>
+            <axis xyz="0 1 0"/>
+            <mimic joint="${prefix}joint_2" multiplier="1"/>
+            <limit lower="${radians(-113)}" upper="${radians(61)}" velocity="1.69" effort="0"/>
+        </joint>
         <!-- Balancer B parallell to Link U -->
         <joint name="${prefix}balancer_B" type="revolute">
-            <parent link="${prefix}link_1"/>
+            <parent link="${prefix}fakelink"/>
             <child link="${prefix}balancer_B"/>
-            <origin xyz="0.400 -0.100 0.7555" rpy="0 0 0" />
+            <!-- <origin xyz="0.000 -0.104 0.000" rpy="0 0 0" /> -->
+            <origin xyz="0.000 -0.100 0.000" rpy="0 0 0" />
             <axis xyz="0 -1 0" />
             <mimic joint="${prefix}joint_3" multiplier="1.0"/>
             <limit lower="${radians(-113)}" upper="${radians(61)}" velocity="1.69" effort="0"/>
-        </joint>
-        <!-- Fakelinke for Balancer A -->
-        <joint name="${prefix}fakelinkA_to_BalancerA" type="revolute">
-            <parent link="${prefix}link_3"/>
-            <child link="${prefix}fakelinkA"/>
-            <origin xyz="-0.500 -0.110 0.000" rpy="0 0 0" />
-            <axis xyz="0 1 0" />
-            <mimic joint="${prefix}joint_3" multiplier="1" offset="${radians(0)}"/>
-            <limit lower="${radians(-180)}" upper="${radians(180)}" velocity="1.69" effort="0"/>
         </joint>
         <!-- Balancer A parallell to Link L -->
         <joint name="${prefix}balancer_A" type="revolute">
-            <parent link="${prefix}fakelinkA"/>
+            <parent link="${prefix}balancer_B"/>
             <child link="${prefix}balancer_A"/>
-            <origin xyz="0.000 0.000 0.000" rpy="0 0 0" />
-            <axis xyz="0 1 0" />
-            <mimic joint="${prefix}joint_2" multiplier="1.0"/>
-            <limit lower="${radians(-55)}" upper="${radians(61)}" velocity="1.69" effort="0"/>
-        </joint>
+            <origin xyz="-0.500 0.000 0.000" rpy="0 0 0" />
+            <axis xyz="0 1 0" />
+            <mimic joint="${prefix}joint_3" multiplier="1.0"/>
+            <limit lower="${radians(-55)}" upper="${radians(61)}" velocity="1.69" effort="0"/>
+        </joint>
+        <!-- Balancer A parallell to Link L -->
+        <!-- <joint name="${prefix}balancer_A" type="revolute">
+            <parent link="${prefix}link_3"/>
+            <child link="${prefix}balancer_A"/>
+            <origin xyz="-0.500 -0.110 0.000" rpy="0 0 0" />
+            <axis xyz="0 1 0" />
+            <mimic joint="${prefix}joint_3" multiplier="1.0"/>
+            <limit lower="${radians(-55)}" upper="${radians(61)}" velocity="1.69" effort="0"/>
+        </joint> -->
+        <!-- Balancer B parallell to Link U -->
+        <!-- <joint name="${prefix}balancer_B" type="revolute">
+            <parent link="${prefix}link_2"/>
+            <child link="${prefix}balancer_B"/>
+            <origin xyz="0.000 -0.104 0.000" rpy="0 0 0" />
+            <axis xyz="0 -1 0" />
+            <mimic joint="${prefix}joint_3" multiplier="1.0"/>
+            <limit lower="${radians(-113)}" upper="${radians(61)}" velocity="1.69" effort="0"/>
+        </joint> -->
         <!-- Cylinder Box -->
         <joint name="${prefix}cylinderbox" type="revolute">
